Commit message: Fault with wheels not rendering Propely

File: install/my_robot_description/share/my_robot_description/urdf/common_properties.xacro (robot description, xacro)
@@ -7,3 +7,30 @@
         <color rgba="0.5 0.5 0.5 1"/>
     </material>
+    <xacro:macro name="box_inertia" params="m x y z o_xyz o_rpy">
+        <inertial>
+            <mass value="${m}" />
+            <origin xyz="${o_xyz}" rpy="${o_rpy}" />
+            <inertia ixx="${(m/12)*(y*y+z*z)}" ixy="0" ixz="0"
+                     iyy="${(m/12)*(x*x+z*z)}" iyz="0"
+                     izz="${(m/12)*(y*y+x*x)}" />
+        </inertial>
+    </xacro:macro>
+    <xacro:macro name="cylinder_inertia" params="m x z o_xyz o_rpy">
+        <inertial>
+            <mass value="${m}" />
+            <origin xyz="${o_xyz}" rpy="${o_rpy}" />
+            <inertia ixx="${(m/12)*(3*(x*x)+(z*z))}" ixy="0" ixz="0"
+                     iyy="${(m/12)*(3*(x*x)+(z*z))}" iyz="0"
+                     izz="${(m/2)*(x*x)}"/>
+        </inertial>
+    </xacro:macro>
+    <xacro:macro name="sphere_inertia" params="m x o_xyz o_rpy">
+        <inertial>
+            <mass value="${m}" />
+            <origin xyz="${o_xyz}" rpy="${o_rpy}" />
+            <inertia ixx="${(2*m/5)*(x*x)}" ixy="0" ixz="0"
+                     iyy="${(2*m/5)*(x*x)}" iyz="0"
+                     izz="${(2*m/5)*(x*x)}"/>
+        </inertial>
+    </xacro:macro>
 </robot>

File: install/my_robot_description/share/my_robot_description/urdf/mobile_base.xacro (robot description, xacro)
@@ -1,5 +1,5 @@
 <?xml version="1.0"?>
 <robot xmlns:xacro = "http://www.ros.org/wiki/xacro">
-    <xacro:property name="base_length" value="1.0"/>
+    <xacro:property name="base_length" value="0.6"/>
     <xacro:property name="base_width" value="0.4"/>
     <xacro:property name="base_height" value="0.2"/>
@@ -7,14 +7,4 @@
     <xacro:property name="wheel_length" value="0.05"/>
     <xacro:property name="castor_radius" value="0.05"/>
-    <!-- <xacro:macro name="example_macro" params="a b c">
-        <link name="dummy_link">
-            <visual>
-                <geometry>
-                    <box size="${a} ${b} ${c}" />
-                </geometry>
-            </visual>
-        </link>
-    </xacro:macro>
-    <xacro:example_macro a="2" b="3" c="4"/> -->
     <link name="base_footprint" />
     <link name="base_link">
@@ -26,5 +16,13 @@
             <material name="green">
             </material>
+            <collision>
+                <geometry>
+                    <box size="${base_length} ${base_width} ${base_height}"/>
+                </geometry>
+                <origin xyz="0 0 ${base_height/2.0}" rpy="0 0 0"/>
+            </collision>
         </visual>
+        <xacro:box_inertia m="5.0" x="${base_length}" y="${base_width}" z="${base_height}"
+                            o_xyz="0 0 ${base_height/2.0}" o_rpy="0 0 0"/>
     </link>
     <xacro:macro name="wheel_link" params="suffix">
@@ -38,4 +36,12 @@
                 </material>
             </visual>
+            <collision>
+                <geometry>
+                    <sphere radius="${wheel_radius}" />
+                </geometry>
+                <origin xyz="0 0 0" rpy="0 0 0"/>
+            </collision>
+            <xacro:cylinder_inertia m="1.0" x="${wheel_radius}" z="${wheel_length}"
+                            o_xyz="0 0 0" o_rpy="${pi/2.0} 0 0"/>
         </link>
     </xacro:macro>
@@ -45,5 +51,5 @@
         <visual>
             <geometry>
-                <sphere radius="${castor_radius}" />
+                <sphere radius="${wheel_radius/2.0}" />
             </geometry>
             <origin xyz="0 0 0" rpy="0 0 0"/>
@@ -51,9 +57,22 @@
             </material>
         </visual>
+        <collision>
+            <geometry>
+                <sphere radius="${wheel_radius/2.0}" />
+            </geometry>
+            <origin xyz="0 0 0" rpy="0 0 0"/>
+        </collision>
+        <xacro:sphere_inertia m="0.5" x="${wheel_radius/2}"
+                            o_xyz="0 0 0" o_rpy="0 0 0"/>
     </link>
+    <joint name="base_joint" type="fixed">
+        <parent link="base_footprint" />
+        <child link="base_link" />
+        <origin xyz="0 0 ${wheel_radius}" rpy="0 0 0" />
+    </joint>
     <joint name="my_robot_wheel1" type="continuous">
         <parent link="base_link" />
         <child link="wheel_1" />
-        <origin xyz="${base_length /4.0} ${base_width /2.0} 0" rpy="0 0 0" />
+        <origin xyz="${base_length /4.0} ${(base_width + wheel_length) /2.0} 0" rpy="0 0 0" />
         <axis xyz="0 1 0" />
         <limit effort="100" velocity="100" />
@@ -62,5 +81,5 @@
         <parent link="base_link" />
         <child link="wheel_2" />
-        <origin xyz="${base_length /4.0} ${-base_width /2.0} 0" rpy="0 0 0" />
+        <origin xyz="${base_length /4.0} ${-(base_width + wheel_length) /2.0} 0" rpy="0 0 0" />
         <axis xyz="0 1 0" />
         <limit effort="100" velocity="100" />
@@ -69,10 +88,5 @@
         <parent link="base_link" />
         <child link="castorlink" />
-        <origin xyz="${-base_width /2.0} 0 ${-castor_radius}"/>
-    </joint>
-    <joint name="base_joint" type="fixed">
-        <parent link="base_footprint" />
-        <child link="base_link" />
-        <origin xyz="0 0 -0.1" rpy="0 0 0" />
+        <origin xyz="${-base_length /3.0} 0 ${-wheel_radius/2}"/>
     </joint>
 </robot>

File: install/my_robot_description/share/my_robot_description/urdf/my_robot.urdf.xacro (robot description, xacro)
@@ -3,3 +3,4 @@
     <xacro:include filename="common_properties.xacro"/>
     <xacro:include filename="mobile_base.xacro"/>
+    <xacro:include filename="mobile_base_gazebo.xacro" />
 </robot>

Commit message: Fixed the Data

File: install/my_robot_description/share/my_robot_description/urdf/common_properties.xacro (robot description, xacro)
@@ -1,9 +1,9 @@
 <?xml version="1.0"?>
-<robot xmlns:xacro = "http://www.ros.org/wiki/xacro">
-    <material name="green">
-        <color rgba="0 0.5 0 1"/>
+<robot xmlns:xacro="http://www.ros.org/wiki/xacro">
+    <material name="blue">
+        <color rgba="0 0 0.5 1" />
     </material>
     <material name="grey">
-        <color rgba="0.5 0.5 0.5 1"/>
+        <color rgba="0.5 0.5 0.5 1" />
     </material>
     <xacro:macro name="box_inertia" params="m x y z o_xyz o_rpy">
@@ -11,25 +11,25 @@
             <mass value="${m}" />
             <origin xyz="${o_xyz}" rpy="${o_rpy}" />
-            <inertia ixx="${(m/12)*(y*y+z*z)}" ixy="0" ixz="0"
-                     iyy="${(m/12)*(x*x+z*z)}" iyz="0"
-                     izz="${(m/12)*(y*y+x*x)}" />
+            <inertia ixx="${(m/12) * (y*y + z*z)}" ixy="0" ixz="0"
+                     iyy="${(m/12) * (x*x + z*z)}" iyz="0"
+                     izz="${(m/12) * (x*x + y*y)}" />
         </inertial>
     </xacro:macro>
-    <xacro:macro name="cylinder_inertia" params="m x z o_xyz o_rpy">
+    <xacro:macro name="cylinder_inertia" params="m r l o_xyz o_rpy">
         <inertial>
             <mass value="${m}" />
             <origin xyz="${o_xyz}" rpy="${o_rpy}" />
-            <inertia ixx="${(m/12)*(3*(x*x)+(z*z))}" ixy="0" ixz="0"
-                     iyy="${(m/12)*(3*(x*x)+(z*z))}" iyz="0"
-                     izz="${(m/2)*(x*x)}"/>
+            <inertia ixx="${(m/12) * (3*r*r + l*l)}" ixy="0" ixz="0"
+                     iyy="${(m/12) * (3*r*r + l*l)}" iyz="0"
+                     izz="${(m/2) * (r*r)}" />
         </inertial>
     </xacro:macro>
-    <xacro:macro name="sphere_inertia" params="m x o_xyz o_rpy">
+    <xacro:macro name="sphere_inertia" params="m r o_xyz o_rpy">
         <inertial>
             <mass value="${m}" />
             <origin xyz="${o_xyz}" rpy="${o_rpy}" />
-            <inertia ixx="${(2*m/5)*(x*x)}" ixy="0" ixz="0"
-                     iyy="${(2*m/5)*(x*x)}" iyz="0"
-                     izz="${(2*m/5)*(x*x)}"/>
+            <inertia ixx="${(2/5) * m * r * r}" ixy="0" ixz="0"
+                     iyy="${(2/5) * m * r * r}" iyz="0"
+                     izz="${(2/5) * m * r * r}" />
         </inertial>
     </xacro:macro>

File: install/my_robot_description/share/my_robot_description/urdf/mobile_base.xacro (robot description, xacro)
@@ -1,38 +1,35 @@
 <?xml version="1.0"?>
-<robot xmlns:xacro = "http://www.ros.org/wiki/xacro">
-    <xacro:property name="base_length" value="0.6"/>
-    <xacro:property name="base_width" value="0.4"/>
-    <xacro:property name="base_height" value="0.2"/>
-    <xacro:property name="wheel_radius" value="0.1"/>
-    <xacro:property name="wheel_length" value="0.05"/>
-    <xacro:property name="castor_radius" value="0.05"/>
+<robot xmlns:xacro="http://www.ros.org/wiki/xacro">
+    <xacro:property name="base_length" value="0.6" />
+    <xacro:property name="base_width" value="0.4" />
+    <xacro:property name="base_height" value="0.2" />
+    <xacro:property name="wheel_radius" value="0.1" />
+    <xacro:property name="wheel_length" value="0.05" />
     <link name="base_footprint" />
     <link name="base_link">
         <visual>
             <geometry>
-                <box size="${base_length} ${base_width} ${base_height}"/>
+                <box size="${base_length} ${base_width} ${base_height}" />
             </geometry>
-            <origin xyz="0 0 ${base_height/2.0}" rpy="0 0 0"/>
-            <material name="green">
-            </material>
-            <collision>
-                <geometry>
-                    <box size="${base_length} ${base_width} ${base_height}"/>
-                </geometry>
-                <origin xyz="0 0 ${base_height/2.0}" rpy="0 0 0"/>
-            </collision>
+            <origin xyz="0 0 ${base_height / 2.0}" rpy="0 0 0" />
+            <material name="blue" />
         </visual>
+        <collision>
+            <geometry>
+                <box size="${base_length} ${base_width} ${base_height}" />
+            </geometry>
+            <origin xyz="0 0 ${base_height / 2.0}" rpy="0 0 0" />
+        </collision>
         <xacro:box_inertia m="5.0" x="${base_length}" y="${base_width}" z="${base_height}"
-                            o_xyz="0 0 ${base_height/2.0}" o_rpy="0 0 0"/>
+                           o_xyz="0 0 ${base_height / 2.0}" o_rpy="0 0 0" />
     </link>
-    <xacro:macro name="wheel_link" params="suffix">
-        <link name="wheel_${suffix}">
+    <xacro:macro name="wheel_link" params="prefix">
+        <link name="${prefix}_wheel_link">
             <visual>
                 <geometry>
-                    <cylinder radius="${wheel_radius}" length="${wheel_length}"/>
+                    <cylinder radius="${wheel_radius}" length="${wheel_length}" />
                 </geometry>
-                <origin xyz="0 0 0" rpy="${pi/2.0} 0 0"/>
-                <material name="grey">
-                </material>
+                <origin xyz="0 0 0" rpy="${pi / 2.0} 0 0" />
+                <material name="grey" />
             </visual>
             <collision>
@@ -40,53 +37,50 @@
                     <sphere radius="${wheel_radius}" />
                 </geometry>
-                <origin xyz="0 0 0" rpy="0 0 0"/>
+                <origin xyz="0 0 0" rpy="0 0 0" />
             </collision>
-            <xacro:cylinder_inertia m="1.0" x="${wheel_radius}" z="${wheel_length}"
-                            o_xyz="0 0 0" o_rpy="${pi/2.0} 0 0"/>
+            <xacro:cylinder_inertia m="1.0" r="${wheel_radius}" l="${wheel_length}"
+                                    o_xyz="0 0 0" o_rpy="${pi / 2.0} 0 0" />
         </link>
     </xacro:macro>
-    <xacro:wheel_link suffix="1" />
-    <xacro:wheel_link suffix="2" />
-    <link name="castorlink">
+    <xacro:wheel_link prefix="right" />
+    <xacro:wheel_link prefix="left" />
+    <link name="caster_wheel_link">
         <visual>
             <geometry>
-                <sphere radius="${wheel_radius/2.0}" />
+                <sphere radius="${wheel_radius / 2.0}" />
             </geometry>
-            <origin xyz="0 0 0" rpy="0 0 0"/>
-            <material name="grey">
-            </material>
+            <origin xyz="0 0 0" rpy="0 0 0" />
+            <material name="grey" />
         </visual>
         <collision>
             <geometry>
-                <sphere radius="${wheel_radius/2.0}" />
+                <sphere radius="${wheel_radius / 2.0}" />
             </geometry>
-            <origin xyz="0 0 0" rpy="0 0 0"/>
+            <origin xyz="0 0 0" rpy="0 0 0" />
         </collision>
-        <xacro:sphere_inertia m="0.5" x="${wheel_radius/2}"
-                            o_xyz="0 0 0" o_rpy="0 0 0"/>
+        <xacro:sphere_inertia m="0.5" r="${wheel_radius / 2.0}"
+                              o_xyz="0 0 0" o_rpy="0 0 0" />
     </link>
     <joint name="base_joint" type="fixed">
         <parent link="base_footprint" />
         <child link="base_link" />
-        <origin xyz="0 0 ${wheel_radius}" rpy="0 0 0" />
+        <origin xyz="0 0 ${wheel_radius}" rpy="0 0 0"/>
     </joint>
-    <joint name="my_robot_wheel1" type="continuous">
+    <joint name="base_right_wheel_joint" type="continuous">
         <parent link="base_link" />
-        <child link="wheel_1" />
-        <origin xyz="${base_length /4.0} ${(base_width + wheel_length) /2.0} 0" rpy="0 0 0" />
+        <child link="right_wheel_link" />
+        <origin xyz="${-base_length / 4.0} ${-(base_width + wheel_length) / 2.0} 0" rpy="0 0 0" />
         <axis xyz="0 1 0" />
-        <limit effort="100" velocity="100" />
     </joint>
-    <joint name="my_robot_wheel2" type="continuous">
+    <joint name="base_left_wheel_joint" type="continuous">
         <parent link="base_link" />
-        <child link="wheel_2" />
-        <origin xyz="${base_length /4.0} ${-(base_width + wheel_length) /2.0} 0" rpy="0 0 0" />
+        <child link="left_wheel_link" />
+        <origin xyz="${-base_length / 4.0} ${(base_width + wheel_length) / 2.0} 0" rpy="0 0 0" />
         <axis xyz="0 1 0" />
-        <limit effort="100" velocity="100" />
     </joint>
-    <joint name="my_robot_castor_wheel" type="fixed">
+    <joint name="base_caster_wheel_joint" type="fixed">
         <parent link="base_link" />
-        <child link="castorlink" />
-        <origin xyz="${-base_length /3.0} 0 ${-wheel_radius/2}"/>
+        <child link="caster_wheel_link" />
+        <origin xyz="${base_length / 3.0} 0 ${-wheel_radius / 2.0}" rpy="0 0 0" />
     </joint>
 </robot>

File: install/my_robot_description/share/my_robot_description/urdf/mobile_base_gazebo.xacro (robot description, xacro)
@@ -1,5 +1,5 @@
 <?xml version="1.0"?>
-<robot name="my_robot" xmlns:xacro="http://www.ros.org/wiki/xacro">
-    <gazebo reference="my_robot_castor_wheel">
+<robot xmlns:xacro="http://www.ros.org/wiki/xacro">
+    <gazebo reference="caster_wheel_link">
         <mu1 value="0.1" />
         <mu2 value="0.1" />
@@ -9,10 +9,6 @@
             filename="gz-sim-diff-drive-system"
             name="gz::sim::systems::DiffDrive">
-            <left_joint>
-                my_robot_wheel1
-            </left_joint>
-            <right_joint>
-                my_robot_wheel2
-            </right_joint>
+            <left_joint>base_left_wheel_joint</left_joint>
+            <right_joint>base_right_wheel_joint</right_joint>
             <wheel_separation>0.45</wheel_separation>
             <wheel_radius>0.1</wheel_radius>
@@ -25,6 +21,6 @@
             filename="gz-sim-joint-state-publisher-system"
             name="gz::sim::systems::JointStatePublisher">
-            <joint_name>my_robot_wheel1</joint_name>
-            <joint_name>my_robot_wheel2</joint_name>
+            <joint_name>base_left_wheel_joint</joint_name>
+            <joint_name>base_right_wheel_joint</joint_name>
         </plugin>
     </gazebo>
